Commit message: Add files via upload

File: tag.urdf (robot description, URDF)
Before this commit: robot artag, 0 links, 0 joints
Links:
- added link tag_background_link, mass 0.01; collision box size=0.1 0.1 0.0001; visual box size=0.1 0.1 0.001
- added link tag_link, mass 0.01; collision mesh filename=package://vigir_ar_alvar_description/meshes/tag.dae; visual mesh filename=package://vigir_ar_alvar_description/meshes/tag.dae
Joints:
- added joint tag_background_joint: type fixed, parent tag_link, child tag_background_link, origin xyz=0 0 -0.001 rpy=0 0 0
- added joint tag_joint: type fixed, parent base_link, child tag_link, origin xyz=0.7 0.0 0.0 rpy=0 0 0
