Commit message: Add files via upload

File: iRobot_tag.urdf (robot description, URDF)
Before this commit: robot iRobot, 13 links, 12 joints
Links:
- link tag_link: geometry collision mesh filename=/home/oli/tesi_software/Firmare/Tools/sitl_gazebo/models/ta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; visual mesh filename=/home/oli/tesi_software/Firmare/Tools/sitl_gazebo/models/ta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
Joints:
- joint tag_joint: origin xyz=0.0 0.0 0.7 rpy=0 0 0 -> xyz=0.0 0.0 0.18 rpy=0 1.57079632679 0

File: iRobot_tag.xacro (robot description, xacro)
@@ -13,5 +13,5 @@
         <xacro:include filename="${tag_description_dir}/urdf/tag.xacro"/>
     	<xacro:artag name="tag" parent="base_link">
-	  <origin xyz="0.0 0.0 0.7" rpy="0 0 0"/>
+	  <origin xyz="0.0 0.0 0.7" rpy="0 ${pi/2} 0"/>
     	</xacro:artag>
 </robot>

File: iris_base.xacro (robot description, xacro)
@@ -4,10 +4,12 @@
   Is there a reason not to make all properties arguments?
   -->
-  <xacro:arg name='enable_ground_truth' default='false' />
-  <xacro:arg name='enable_mavlink_interface' default='true' />
-  <xacro:arg name='enable_wind' default='false' />
+  <xacro:arg name='name' default='iris' />
   <xacro:arg name='mavlink_addr' default='INADDR_ANY' />
   <xacro:arg name='mavlink_udp_port' default='14560' />
   <xacro:arg name='visual_material' default='DarkGrey' />
+  <xacro:arg name='enable_mavlink_interface' default='true' />
+  <xacro:arg name='enable_wind' default='false' />
+  <!-- The following causes segfault with multiple vehicles if defaults to true!!! -->
+  <xacro:arg name='enable_ground_truth' default='false' />
   <xacro:arg name='enable_logging' default='false' />
   <xacro:arg name='log_file' default='iris' />
