Commit message: Add files via upload
iris_camera_xacro è stata cambiata facendo ruotare la camera di un angolo di 16.5 gradi cioè 0.29 radianti.

File: iris_camera.urdf (robot description, URDF)
Before this commit: robot iris_camera, 12 links, 11 joints
Links:
- link base_link_inertia: geometry collision box size=0.47 0.47 0.11; visual mesh filename=/home/oli/tesi_software/Firmware/Tools/sitl_gazebo/models/r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 scale=1 1 1
- link camera_link: mass 0 -> 0.200; geometry collision mesh filename=/home/oli/tesi_software/Firmware/Tools/sitl_gazebo/models/c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; visual mesh filename=/home/oli/tesi_software/Firmware/Tools/sitl_gazebo/models/c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
- link rotor_0: geometry collision cylinder length=0.005 radius=0.128; visual mesh filename=/home/oli/tesi_software/Firmware/Tools/sitl_gazebo/models/r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 scale=1 1 1
- link rotor_1: geometry collision cylinder length=0.005 radius=0.128; visual mesh filename=/home/oli/tesi_software/Firmware/Tools/sitl_gazebo/models/r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 scale=1 1 1
- link rotor_2: geometry collision cylinder length=0.005 radius=0.128; visual mesh filename=/home/oli/tesi_software/Firmware/Tools/sitl_gazebo/models/r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 scale=1 1 1
- link rotor_3: geometry collision cylinder length=0.005 radius=0.128; visual mesh filename=/home/oli/tesi_software/Firmware/Tools/sitl_gazebo/models/r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 scale=1 1 1
Joints:
- joint camera_joint: origin xyz=0.1475 0.0 0.0 rpy=0 0 0 -> xyz=0.1475 0.0 0.0 rpy=0 0.29 0

File: iris_camera.xacro (robot description, xacro)
@@ -7,5 +7,5 @@
 	<xacro:include filename="$(arg camera_description_dir)/urdf/asus_camera.xacro"/>
     	<xacro:asus_camera name="camera" parent="base_link">
-	  <origin xyz="0.1475 0.0 0.0" rpy="0 0 0"/>
+	  <origin xyz="0.1475 0.0 0.0" rpy="0 0.29 0"/>
     	</xacro:asus_camera>
 </robot>
